File: TestProjects/Test1/Test1.kicad_pcb (KiCad board)
At the start: 2 copper layers, 40 x 46.4 mm, 28 parts, among them J1 Input, SW1 SW_DIP_x08, U1 74AHC244

Commit message: feat: auto-exclude and refill copper fill zones (v0.20.0)
Zones with `(fill yes ...)` are now handled correctly end-to-end:
- `pcb._parse_zones` records `fill_enabled` on each zone dict
- `pcb.zone_fill_nets(board)` returns nets that have an active pour
- `pcb.try_refill_zones(path)` calls kicad-cli to regenerate the pour
- `geometry.board_obstacles` skips fill zones (not routing obstacles)
- CLI and GUI pipelines auto-exclude fill nets from routing/placement
  and call try_refill_zones after writing the output board
- Added GND B.Cu fill zone to Test1.kicad_pcb
- 4 new unit tests covering parsing, zone_fill_nets, and obstacle skip

Co-Authored-By: Claude Sonnet 4.6 <noreply@anthropic.com>
Routing:
- added copper zone on B.Cu, net GND
Changed lines of the file:
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@@
 	)
 	(embedded_fonts no)
+	(zone
+		(net "GND")
+		(layer "B.Cu")
+		(hatch edge 0.5)
+		(connect_pads (clearance 0.5))
+		(min_thickness 0.25)
+		(fill yes (thermal_gap 0.5) (thermal_bridge_width 0.5) (island_removal_mode 0))
+		(polygon
+			(pts
+				(xy 39 37) (xy 77.54296 37.03724) (xy 77.5 81.5)
+				(xy 43.088185 81.937418) (xy 42.907907 67.754942) (xy 38.5 65)
+			)
+		)
+	)
 )
