File: TestProjects/Test1/Test1.kicad_pcb (KiCad board)
At the start: 2 copper layers, 40 x 46.4 mm, 28 parts, among them J1 Input, SW1 SW_DIP_x08, U1 74AHC244

Commit message: Added fill to test1 board.
Routing:
- net Net-(J1-Pin_9): vias 2 -> 0
- net Net-(J1-Pin_6): vias 2 -> 0
- net Net-(D8-A): vias 1 -> 0
- net Net-(D7-A): vias 1 -> 0
- net Net-(D6-A): vias 1 -> 0
- net Net-(D5-A): vias 1 -> 0
- net Net-(D4-A): vias 1 -> 0
- net 5V: vias 1 -> 0
- added copper zone on B.Cu, net GND
Changed lines of the file:
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@@
 	)
 	(footprint "Connector_PinHeader_2.54mm:PinHeader_1x10_P2.54mm_Vertical"
+		(locked yes)
 		(layer "F.Cu")
 		(at 40.5 41)
@@
 	)
 	(gr_text "D. Q. McDonald\nv1.0 May 2026"
+		(locked yes)
 		(at 60 71 0)
 		(layer "F.SilkS")
@@
 	)
 	(gr_text "Bus Indicator"
+		(locked yes)
 		(at 60 40 0)
 		(layer "F.SilkS")
@@
 		)
 	)
-	(via
-		(at 62.2181 61.69)
-		(size 0.6)
-		(drill 0.3)
-		(layers "F.Cu" "B.Cu")
-		(net "Net-(D4-A)")
-	)
-	(via
-		(at 64.3689 57.6051)
-		(size 0.6)
-		(drill 0.3)
-		(layers "F.Cu" "B.Cu")
-		(net "Net-(D6-A)")
-	)
-	(via
-		(at 64.5577 53.6468)
-		(size 0.6)
-		(drill 0.3)
-		(layers "F.Cu" "B.Cu")
-		(net "Net-(D5-A)")
-	)
-	(via
-		(at 64.4765 73.0447)
-		(size 0.6)
-		(drill 0.3)
-		(layers "F.Cu" "B.Cu")
-		(net "Net-(J1-Pin_6)")
-	)
-	(via
-		(at 52.0588 64.0316)
-		(size 0.6)
-		(drill 0.3)
-		(layers "F.Cu" "B.Cu")
-		(net "Net-(J1-Pin_6)")
-	)
-	(via
-		(at 64.4008 60.2211)
-		(size 0.6)
-		(drill 0.3)
-		(layers "F.Cu" "B.Cu")
-		(net "Net-(D7-A)")
-	)
-	(via
-		(at 75.0045 58.2239)
-		(size 0.6)
-		(drill 0.3)
-		(layers "F.Cu" "B.Cu")
-		(net "5V")
-	)
-	(via
-		(at 40.5 67.0276)
-		(size 0.6)
-		(drill 0.3)
-		(layers "F.Cu" "B.Cu")
-		(net "Net-(J1-Pin_9)")
-	)
-	(via
-		(at 44.6 72)
-		(size 0.6)
-		(drill 0.3)
-		(layers "F.Cu" "B.Cu")
-		(net "Net-(J1-Pin_9)")
-	)
-	(via
-		(at 64.5029 62.9312)
-		(size 0.6)
-		(drill 0.3)
-		(layers "F.Cu" "B.Cu")
-		(net "Net-(D8-A)")
+	(zone
+		(net "GND")
+		(layer "B.Cu")
+		(hatch edge 0.5)
+		(connect_pads
+			(clearance 0.5)
+		)
+		(min_thickness 0.25)
+		(fill yes
+			(thermal_gap 0.5)
+			(thermal_bridge_width 0.5)
+			(island_removal_mode 0)
+		)
+		(polygon
+			(pts
+				(xy 39 37) (xy 77.54296 37.03724) (xy 77.5 81.5) (xy 43.088185 81.937418) (xy 42.907907 67.754942)
+				(xy 38.5 65)
+			)
+		)
 	)
 	(embedded_fonts no)
