File: TestProjects/Test2/Test2.kicad_pcb (KiCad board)
At the start: 2 copper layers, 23.5 x 21.5 mm, 4 parts, among them SW1 SW_Push

Commit message: fix(lint): resolve pylint warnings and E-level errors
- Remove unused imports: re (netlist), strings (autoroute), simpledialog (gui)
- Fix cell-var-from-loop in netlist (lambda default arg) and pipeline (closures)
- Fix reimported time in autoroute (use top-level import directly)
- Drop unused variable: keep_outline (autoroute), layers_p (report)
- Rename shadowing local: field -> cfield in placement._congestion_sum
- Type CycleHooks callbacks as Callable|None (fixes E1102 not-callable)
- Add Callable import to pipeline
- Convert RunConfig to @dataclass (fixes 39 E1101 no-member false positives
  from __slots__ + dynamic setattr pattern)
- Suppress intentional dangerous-default-value in cycle timer closures
- Mark probe imports in gui/__init__ with pylint disable
- Fix unused tip variable in gui/app.py metrics panel loop

Score: 8.88 -> 9.23/10

Co-Authored-By: Claude Sonnet 4.6 <noreply@anthropic.com>
Routing:
- net Net-(BT1-+): track 0.00 -> 8.47 mm
- net Net-(D1-A): track 0.00 -> 7.94 mm
- net Net-(BT1--): track 0.00 -> 7.15 mm
- net Net-(D1-K): track 0.00 -> 6.74 mm
Changed lines of the file:
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@@
 		(title "Test Board for Autorouter")
 		(date "2026-05-27")
+		(comment 1 "PyAutoRoute v0.41.0 — routed 2026-06-03")
+		(comment 2 "PyAutoRoute v0.41.0 — routed 2026-06-03")
 	)
 	(layers
@@
 	)
 	(embedded_fonts no)
+	(segment
+		(start 68.6 61.099999999999994)
+		(end 64.7 57.2)
+		(width 0.2)
+		(layer "F.Cu")
+		(net "Net-(BT1--)")
+	)
+	(segment
+		(start 64.7 57.2)
+		(end 64.4 57.2)
+		(width 0.2)
+		(layer "F.Cu")
+		(net "Net-(BT1--)")
+	)
+	(segment
+		(start 69 61.5)
+		(end 68.6 61.099999999999994)
+		(width 0.2)
+		(layer "F.Cu")
+		(net "Net-(BT1--)")
+	)
+	(segment
+		(start 64 56.54)
+		(end 64.4 57.2)
+		(width 0.2)
+		(layer "F.Cu")
+		(net "Net-(BT1--)")
+	)
+	(segment
+		(start 74.6 61.099999999999994)
+		(end 76.7 59)
+		(width 0.2)
+		(layer "F.Cu")
+		(net "Net-(D1-K)")
+	)
+	(segment
+		(start 76.7 59)
+		(end 76.7 56.9)
+		(width 0.2)
+		(layer "F.Cu")
+		(net "Net-(D1-K)")
+	)
+	(segment
+		(start 74.08 61.5)
+		(end 74.6 61.099999999999994)
+		(width 0.2)
+		(layer "F.Cu")
+		(net "Net-(D1-K)")
+	)
+	(segment
+		(start 77.5 56.27)
+		(end 76.7 56.9)
+		(width 0.2)
+		(layer "F.Cu")
+		(net "Net-(D1-K)")
+	)
+	(segment
+		(start 77 53)
+		(end 73.4 49.4)
+		(width 0.2)
+		(layer "F.Cu")
+		(net "Net-(D1-A)")
+	)
+	(segment
+		(start 73.4 49.4)
+		(end 73.4 48.2)
+		(width 0.2)
+		(layer "F.Cu")
+		(net "Net-(D1-A)")
+	)
+	(segment
+		(start 77.5 53.730000000000004)
+		(end 77 53)
+		(width 0.2)
+		(layer "F.Cu")
+		(net "Net-(D1-A)")
+	)
+	(segment
+		(start 73.1 47.5)
+		(end 73.4 48.2)
+		(width 0.2)
+		(layer "F.Cu")
+		(net "Net-(D1-A)")
+	)
+	(segment
+		(start 68.6 48.2)
+		(end 64.7 52.1)
+		(width 0.2)
+		(layer "F.Cu")
+		(net "Net-(BT1-+)")
+	)
+	(segment
+		(start 64.7 52.1)
+		(end 64.7 53.3)
+		(width 0.2)
+		(layer "F.Cu")
+		(net "Net-(BT1-+)")
+	)
+	(segment
+		(start 68.9 47.5)
+		(end 68.6 48.2)
+		(width 0.2)
+		(layer "F.Cu")
+		(net "Net-(BT1-+)")
+	)
+	(segment
+		(start 64 54)
+		(end 64.7 53.3)
+		(width 0.2)
+		(layer "F.Cu")
+		(net "Net-(BT1-+)")
+	)
 )
